File: PCB/servo tester.kicad_pcb (KiCad board)
At the start: 2 copper layers, 4 parts

Commit message: done a quite a bit of PCB
Parts:
- removed MainON/OFF1, SweepMode1: SW_Push, Button_Switch_THT:SW_PUSH_6mm_H13mm
- removed RV1: R_Potentiometer, Potentiometer_THT:Potentiometer_Alps_RK09Y11_Single_Horizontal
- added B+1: TestPoint, Connector_Wire:SolderWire-0.75sqmm_1x01_D1.25mm_OD2.3mm, F.Cu at (48.0, 71.3)
- added B-1: TestPoint, Connector_Wire:SolderWire-0.75sqmm_1x01_D1.25mm_OD2.3mm, F.Cu at (48.0, 76.0)
- added P_GND1: TestPoint, Connector_Wire:SolderWire-0.75sqmm_1x01_D1.25mm_OD2.3mm, F.Cu at (103.9, 109.8)
- added P_HIGH1: TestPoint, Connector_Wire:SolderWire-0.75sqmm_1x01_D1.25mm_OD2.3mm, F.Cu at (98.0, 104.3)
- added P_RESIS1: TestPoint, Connector_Wire:SolderWire-0.75sqmm_1x01_D1.25mm_OD2.3mm, F.Cu at (98.0, 111.5)
- added SDA1: TestPoint, Connector_Wire:SolderWire-0.75sqmm_1x01_D1.25mm_OD2.3mm, F.Cu at (91.5, 120.0)
- added SDA2: TestPoint, Connector_Wire:SolderWire-0.75sqmm_1x01_D1.25mm_OD2.3mm, F.Cu at (91.5, 113.0)
- added SW2: SW_Push, Button_Switch_THT:SW_PUSH_6mm_H4.3mm, F.Cu at (60.5, 93.0)
- added SWEEPMODE1: SW_Push, Button_Switch_THT:SW_PUSH_6mm_H4.3mm, F.Cu at (60.8, 107.2)
- added U1: ER_OLEDM0.91_1x-I2C, Display:ER_OLEDM0.91_1x-I2C, F.Cu at (102.7, 69.0)
- added main1: TestPoint, Connector_Wire:SolderWire-0.75sqmm_1x01_D1.25mm_OD2.3mm, F.Cu at (60.0, 71.5)
- added main2: TestPoint, Connector_Wire:SolderWire-0.75sqmm_1x01_D1.25mm_OD2.3mm, F.Cu at (64.7, 71.5)
- A1: value Arduino_Nano_v2.x -> Arduino_Nano_v3.x
- moved A1 36.8 mm to (77.6, 68.6)
Connections:
- A1 pad 1: SERVO1 -> unconnected-(A1-D1/TX-Pad1)
- A1 pad 10: unconnected-(A1-D7-Pad10) -> Net-(A1-D7)
- A1 pad 11: unconnected-(A1-D8-Pad11) -> Net-(A1-D8)
- A1 pad 15: Net-(A1-D12) -> unconnected-(A1-D12-Pad15)
- A1 pad 16: Net-(A1-D13) -> unconnected-(A1-D13-Pad16)
- A1 pad 22: Net-(A1-A3) -> unconnected-(A1-A3-Pad22)
- A1 pad 24: unconnected-(A1-A5-Pad24) -> Net-(A1-A5)
- A1 pad 25: unconnected-(A1-A6-Pad25) -> Net-(A1-A6)
- A1 pad 26: unconnected-(A1-A7-Pad26) -> Net-(A1-A7)
- A1 pad 27: unconnected-(A1-+5V-Pad27) -> Net-(A1-+5V)
- A1 pad 5: SERVO2 -> unconnected-(A1-D2-Pad5)
- A1 pad 6: SERVO3 -> Net-(A1-D3)
- A1 pad 7: unconnected-(A1-D4-Pad7) -> Net-(A1-D4)
Routing:
- net Net-(A1-A5): track 0.00 -> 104.3 mm
- net Net-(U1-SDA): track 0.00 -> 68.7 mm
- net GND: track 0.00 -> 40.9 mm
- net Net-(A1-VIN): track 0.00 -> 33.8 mm
- net Net-(A1-A6): track 0.00 -> 33.0 mm
- net Net-(A1-A4): track 0.00 -> 30.5 mm
- net Net-(A1-D8): track 0.00 -> 28.6 mm
- net Net-(A1-D7): track 0.00 -> 27.8 mm
- net Net-(A1-A7): track 0.00 -> 27.8 mm
- net Net-(A1-D4): track 0.00 -> 27.4 mm
- net Net-(A1-D3): track 0.00 -> 26.5 mm
- net Net-(A1-+5V): track 0.00 -> 15.9 mm
- net Net-(B+1-Pad1): track 0.00 -> 12.1 mm
- added copper zone on B.Cu, net GND
Other:
- board outline added: 75 x 65 mm
- board text added: "SERVO TESTER V1"
- board text added: "VEX7FAR"

Commit message: redid pcb
Parts:
- removed B+1, B-1, P_GND1, P_HIGH1, P_RESIS1, SDA1, SDA2, main1, main2: TestPoint, Connector_Wire:SolderWire-0.75sqmm_1x01_D1.25mm_OD2.3mm
- removed SW2, SWEEPMODE1: SW_Push, Button_Switch_THT:SW_PUSH_6mm_H4.3mm
- added +B1: TestPoint, Connector_Wire:SolderWire-0.5sqmm_1x01_D0.9mm_OD2.1mm, F.Cu at (17.0, 27.0)
- added -B1: TestPoint, Connector_Wire:SolderWire-0.5sqmm_1x01_D0.9mm_OD2.1mm, F.Cu at (17.0, 16.5)
- added B10K1: R_Potentiometer, Potentiometer_THT:Potentiometer_Bourns_3386C_Horizontal, F.Cu at (95.5, 39.0)
- added D4: D, Diode_THT:D_A-405_P10.16mm_Horizontal, F.Cu at (25.9, 35.5)
- added D5: D, Diode_THT:D_A-405_P10.16mm_Horizontal, F.Cu at (70.6, 60.0)
- added S1: Conn_01x01_Pin, Connector_PinHeader_2.54mm:PinHeader_1x01_P2.54mm_Horizontal, F.Cu at (121.6, 51.9)
- added S2: Conn_01x01_Pin, Connector_PinHeader_2.54mm:PinHeader_1x01_P2.54mm_Horizontal, F.Cu at (121.6, 56.5)
- added S3: Conn_01x01_Pin, Connector_PinHeader_2.54mm:PinHeader_1x01_P2.54mm_Horizontal, F.Cu at (121.6, 61.1)
- added SW3: SW_Push, Button_Switch_THT:SW_PUSH_6mm, F.Cu at (73.2, 49.8)
- added SWEEP_TOGGLE1: SW_Push, Button_Switch_THT:SW_PUSH_6mm, F.Cu at (27.8, 54.8)
- added SW_MAIN1: SW_Push, Button_Switch_THT:SW_DIP_SPSTx01_Slide_9.78x4.72mm_W7.62mm_P2.54mm, F.Cu at (31.8, 22.0)
- moved A1 57.9 mm to (41.9, 22.9)
- moved U1 53.7 mm to (66.5, 29.3), turned to 90 degrees
Connections:
- A1 pad 14: unconnected-(A1-D11-Pad14) -> Net-(A1-D11)
- A1 pad 19: unconnected-(A1-A0-Pad19) -> Net-(A1-A0)
- A1 pad 25: Net-(A1-A6) -> unconnected-(A1-A6-Pad25)
- A1 pad 26: Net-(A1-A7) -> unconnected-(A1-A7-Pad26)
- U1 pad 4: Net-(U1-SDA) -> Net-(A1-A4)
Routing:
- net Net-(A1-D11): track 0.00 -> 120.8 mm
- net Net-(A1-A5): track 104.3 -> 22.5 mm
- net Net-(U1-SDA): track 68.7 -> 0.00 mm
- net GND: track 40.9 -> 0.00 mm
- net Net-(A1-A0): track 0.00 -> 40.8 mm
- net Net-(A1-+5V): track 15.9 -> 56.5 mm
- net Net-(A1-A6): track 33.0 -> 0.00 mm
- net Net-(A1-A7): track 27.8 -> 0.00 mm
- net Net-(A1-D8): track 28.6 -> 53.3 mm
- net Net-(D4-K): track 0.00 -> 22.0 mm
- net Net-(A1-D3): track 26.5 -> 5.87 mm
- net Net-(D5-K): track 0.00 -> 13.4 mm
- net Net-(B+1-Pad1): track 12.1 -> 0.00 mm
- net Net-(+B1-Pad1): track 0.00 -> 10.4 mm
- net Net-(A1-VIN): track 33.8 -> 27.4 mm
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Other:
- board size 75 x 65 mm -> 113 x 59 mm

Commit message: finsihed cad
Parts:
- added S1-G1: Conn_01x01_Pin, Connector_PinHeader_2.54mm:PinHeader_1x01_P2.54mm_Horizontal, F.Cu at (122.1, 16.5)
- added S1-P1: Conn_01x01_Pin, Connector_PinHeader_2.54mm:PinHeader_1x01_P2.54mm_Horizontal, F.Cu at (122.1, 27.5)
- added S2-G1: Conn_01x01_Pin, Connector_PinHeader_2.54mm:PinHeader_1x01_P2.54mm_Horizontal, F.Cu at (122.1, 35.5)
- added S2-P1: Conn_01x01_Pin, Connector_PinHeader_2.54mm:PinHeader_1x01_P2.54mm_Horizontal, F.Cu at (122.1, 46.5)
- added S3-G1: Conn_01x01_Pin, Connector_PinHeader_2.54mm:PinHeader_1x01_P2.54mm_Horizontal, F.Cu at (122.1, 54.5)
- added S3-P1: Conn_01x01_Pin, Connector_PinHeader_2.54mm:PinHeader_1x01_P2.54mm_Horizontal, F.Cu at (122.1, 66.0)
- added SB-GND1: Conn_01x01_Pin, Connector_PinHeader_2.54mm:PinHeader_1x01_P2.54mm_Horizontal, F.Cu at (107.5, 11.5)
- added SB-VCC1: Conn_01x01_Pin, Connector_PinHeader_2.54mm:PinHeader_1x01_P2.54mm_Horizontal, F.Cu at (114.5, 11.5)
- moved S1-S1 29.9 mm to (122.1, 22.0)
- moved S2-S1 15.5 mm to (122.1, 41.0)
- moved S3-S1 1.20 mm to (122.1, 60.0)
- renumbered S1 to S1-S1, S2 to S2-S1, S3 to S3-S1
Routing:
- net Net-(S1-P1-Pin_1): track 0.00 -> 70.5 mm
- net Net-(A1-D11): track 120.8 -> 132.4 mm
Other:
- board size 113 x 59 mm -> 113 x 62.5 mm

Commit message: almost ship ready
Parts:
- moved D5 1.00 mm to (71.6, 60.0)
- renumbered SWEEP_TOGGLE1 to MODE1, SW3 to RESET1
